File: hardware/ASDR.sch (KiCad schematic (older format))
At the start: 34 parts

Commit message: schematic done
Parts:
- removed D_CV, EOA, EOR, In, OUT, R_CV, S_CV: PJ301M-12, symbol EURO_CAD:PJ301M-12
- removed P_D, P_DCV, P_R, P_RCV, P_S, P_SCV: R_POT, symbol Device:R_POT
- removed R? (x8): R, symbol Device:R
- removed U? (x3): TLV9004xRUCR, Package_DFN_QFN:Texas_S-PX2QFN-14, symbol Amplifier_Operational:TLV9004xRUCR
- added 100n, 47u: C, symbol Device:C
- added C2, C3: 100n, symbol Device:C
- added C4: 10n, symbol Device:C
- added C?: 47u, symbol Device:C
- added CV_D1, CV_R1, CV_S1, CV_cA1, CV_cD1, CV_cR1, CV_cS1, I_GATE1, I_RETRIG1, I_TRIG1, OUT+1, OUT-1, O_EOA1, O_EOR1: PJ301M-12, symbol Connector:AudioJack2_SwitchT
- added D1, D2: 1N53xxB, Diode_THT:D_DO-201_P15.24mm_Horizontal, symbol Diode:1N53xxB
- added D4: LED, symbol Device:LED
- added D? (x3): D, symbol Device:D
- added J?: Conn_02x05_Counter_Clockwise, symbol Connector_Generic:Conn_02x05_Counter_Clockwise
- added P_D1, P_DCV1, P_R1, P_RCV1, P_S1, P_SCV1, P_cA1, P_cACV1, P_cD1, P_cDCV1, P_cR1, P_cRCV1, P_cS1, P_cSCV1: 100k, symbol Device:R_POT
- added R1, R10, R11, R12, R13, R14, R15, R17, R19, R21, R23, R24, R25, R26, R28, R3, R32, R33, R34, R5, R7, R9: 100k, symbol Device:R
- added R16, R18, R2, R20, R22, R4, R6, R8: 180k, symbol Device:R
- added R27: 1.5k, symbol Device:R
- added R29, R30: 200, symbol Device:R
- added R?: 1k, symbol Device:R
- added U2, U?: TL074, symbol Amplifier_Operational:TL074
- added U3, U4, U5, U6, U7, U8, U9: TLV9004xRUCR, Package_DFN_QFN:Texas_S-PX2QFN-14, symbol Amplifier_Operational:TLV9004xRUCR
- added U?: LM1117-5.0, symbol Regulator_Linear:LM1117-5.0
- C1: renamed from C?; value 10n -> 100n
- CV_A1: renamed from A_CV; symbol EURO_CAD:PJ301M-12 -> Connector:AudioJack2_SwitchT
- P_A1: renamed from P_A; value R_POT -> 100k
- P_ACV1: renamed from P_ACV; value R_POT -> 100k
- gave numbers to parts that had none: 5
Connections:
- net +5V: now also 100n.1, 47u.1, C3.1, R9.2, U3.3 (V+), U?.2 (VO); no longer P_A1.3
- net GND: now also CV_A1.S, CV_A1.TN, P_A1.3, U1.2 (+), 100n.2, 47u.2, C3.2, C4.2, C?.2, CV_D1.S, CV_D1.TN, CV_R1.S, CV_R1.TN, CV_S1.S, CV_S1.TN, CV_cA1.S, CV_cA1.TN, CV_cD1.S, CV_cD1.TN, CV_cR1.S, CV_cR1.TN, CV_cS1.S, CV_cS1.TN, D1.2 (A), D2.2 (A), I_GATE1.S, I_RETRIG1.S, I_TRIG1.S, J?.2 (Pin_2), J?.3 (Pin_3), J?.4 (Pin_4), J?.7 (Pin_7), J?.8 (Pin_8), J?.9 (Pin_9), OUT+1.S, OUT-1.S, O_EOA1.S, O_EOR1.S, P_D1.3, P_DCV1.1, P_R1.3, P_RCV1.1, P_S1.3, P_SCV1.1, P_cA1.3, P_cACV1.1, P_cD1.3, P_cDCV1.1, P_cR1.3, P_cRCV1.1, P_cS1.3, P_cSCV1.1, R32.1, U2.10 (+), U2.5 (+), U3.10 (V-), U3.2 (+), U4.2 (+), U5.2 (+), U6.2 (+), U7.2 (+), U8.2 (+), U9.2 (+), U?.1 (GND), U?.12 (+); no longer CV_A1.1, CV_A1.2, P_A1.1
- net GATE: now reaches A1.10 (D7)
- net GATE: now also D3.1 (K), R31.2
- net at A1.12 (D9): now also O_EOR1.T
- net at A1.13 (D10): now also O_EOA1.T
- net A: now reaches A1.19 (A0), U1.14
- net A: now also R10.1; no longer U1.1 (-)
- net D: now reaches A1.20 (A1)
- net D: now also R11.1, U3.14
- net S: now reaches A1.21 (A2)
- net S: now also R12.1, U4.14
- net R: now reaches A1.22 (A3)
- net R: now also R13.1, U5.14
- net cA: now reaches A1.23 (SDA/A4)
- net cA: now also R23.1, U6.14
- net cD: now reaches A1.24 (SCL/A5)
- net cD: now also R24.1, U7.14
- net cS: now reaches A1.25 (A6)
- net cS: now also R25.1, U8.14
- net cR: now reaches A1.26 (A7)
- net cR: now also R26.1, U9.14
- net at A1.6 (D3): now also D2.1 (K), R30.2
- net at U10.8 (VoutA): now also R27.2
- net at P_ACV1.2: now also R2.2
- net at P_A1.2: now also R1.2
- net at R31.1: now also I_GATE1.T
- net at P_ACV1.3: now also CV_A1.T; no longer CV_A1.3
- new net: A1.5 (D2), D1.1 (K), R29.2
- new net: R1.1, R10.2, R2.1, U1.1 (-)
- new net: OUT+1.T, R28.2, R34.1, R?.2, U2.1
- new net: R32.2, R34.2, U2.2 (-)
- new net: C4.1, R27.1, U2.3 (+)
- new net: R28.1, R33.2, U2.6 (-)
- new net: OUT-1.T, R33.1, U2.7
- new net: D4.1 (K), D?.2 (A), U?.14
- new net: D4.2 (A), D?.1 (K), R?.1, U?.13 (-)
- new net: CV_D1.T, P_DCV1.3
- new net: P_DCV1.2, R4.2
- new net: P_D1.2, R3.2
- new net: R11.2, R3.1, R4.1, U3.1 (-)
- new net: CV_S1.T, P_SCV1.3
- new net: P_SCV1.2, R6.2
- new net: P_S1.2, R5.2
- new net: R12.2, R5.1, R6.1, U4.1 (-)
- new net: CV_R1.T, P_RCV1.3
- new net: P_RCV1.2, R8.2
- new net: P_R1.2, R7.2
- new net: R13.2, R7.1, R8.1, U5.1 (-)
- new net: C?.1, D?.2 (A), J?.1 (Pin_1), J?.10 (Pin_10), U?.3 (VI)
- new net: D?.1 (K), J?.5 (Pin_5), J?.6 (Pin_6)
- new net: R14.2, R9.1, U2.9 (-)
- new net: I_RETRIG1.T, R30.1
- new net: I_TRIG1.T, R29.1
- new net: CV_cA1.T, P_cACV1.3
- new net: P_cACV1.2, R16.2
- new net: P_cA1.2, R15.2
- new net: R15.1, R16.1, R23.2, U6.1 (-)
- new net: CV_cD1.T, P_cDCV1.3
- new net: P_cDCV1.2, R18.2
- new net: P_cD1.2, R17.2
- new net: R17.1, R18.1, R24.2, U7.1 (-)
- new net: CV_cS1.T, P_cSCV1.3
- new net: P_cSCV1.2, R20.2
- new net: P_cS1.2, R19.2
- new net: R19.1, R20.1, R25.2, U8.1 (-)
- new net: CV_cR1.T, P_cRCV1.3
- new net: P_cRCV1.2, R22.2
- new net: P_cR1.2, R21.2
- new net: R21.1, R22.1, R26.2, U9.1 (-)
- new net +12V: C2.1, D?.1 (K), U2.4 (V+)
- new net -12V: C2.2, D?.2 (A), U2.11 (V-)
- new net -5V: P_A1.1, P_D1.1, P_R1.1, P_S1.1, P_cA1.1, P_cD1.1, P_cR1.1, P_cS1.1, R14.1, U2.8
Other:
- note added: "11 khz LP\n"
- note added: "INPUT"
- note added: "POWER"
- note added: "[-10; 10] V"
- note added: "[0; -10] V"
- note added: "[0; 10] V"
- note added: "outLED\n"
- moved on the sheet: A1, C1, D3, P_A1, P_ACV1, R31, U10, U1A, U1E
