File: hardware/ADSR.sch (KiCad schematic (older format))
At the start: 87 parts, among them J1 Conn_02x05_Counter_Clockwise, U1 TLV9004xRUCR, U10 MCP4921-EP, U11 LM1117-5.0, U2 TL074, U3 TLV9004xRUCR

Commit message: added TLV9004 to library and placement is final
Parts:
- J1: footprint Connector_PinSocket_2.54mm:PinSocket_2x05_P2.54mm_Vertical -> Connector_PinHeader_2.54mm:PinHeader_2x05_P2.54mm_Vertical; symbol Connector_Generic:Conn_02x05_Counter_Clockwise -> Connector_Generic:Conn_02x05_Odd_Even
- U1, U3: value TLV9004xRUCR -> TLV9004; symbol Amplifier_Operational:TLV9004xRUCR -> ADSR:TLV9004xSOIC
- renumbered C1 to c3, C2 to c4, C3 to c5, C5 to c6, C4 to c7
Connections:
- wire segments 229 -> 233

Commit message: added more puffer caps. im lazy. go autoRoute
Parts:
- added c8, c9: 100n, Capacitor_SMD:C_0805_2012Metric_Pad1.18x1.45mm_HandSolder, symbol Device:C
- c1: value 47u -> 100n; footprint Capacitor_THT:CP_Radial_D5.0mm_P2.50mm -> Capacitor_SMD:C_0805_2012Metric_Pad1.18x1.45mm_HandSolder
Connections:
- wire segments 233 -> 236
Changed lines of the file:
@@
 $EndComp
 Wire Wire Line
-	8500 3950 8500 4050
+	8500 3950 8500 4000
 $Comp
 L power:+5V #PWR062
@@
 	1    0    0    -1
 $EndComp
-Wire Wire Line
-	4200 2100 4350 2100
 $Comp
 L power:+5V #PWR083
@@
 Wire Wire Line
 	3350 2100 3600 2100
-$Comp
-L Device:C c1
-U 1 1 6077CFBB
-P 4350 2250
-F 0 "c1" H 4465 2296 50  0000 L CNN
-F 1 "47u" H 4465 2205 50  0000 L CNN
-F 2 "Capacitor_THT:CP_Radial_D5.0mm_P2.50mm" H 4388 2100 50  0001 C CNN
-F 3 "~" H 4350 2250 50  0001 C CNN
-	1    4350 2250
-	1    0    0    -1
-$EndComp
-Connection ~ 4350 2100
-Wire Wire Line
-	4350 2100 4700 2100
 $Comp
 L Device:C c2
@@
 	1    0    0    1
 $EndComp
+$Comp
+L Device:C c8
+U 1 1 6075567B
+P 6450 3550
+F 0 "c8" H 6565 3596 50  0000 L CNN
+F 1 "100n" H 6565 3505 50  0000 L CNN
+F 2 "Capacitor_SMD:C_0805_2012Metric_Pad1.18x1.45mm_HandSolder" H 6488 3400 50  0001 C CNN
+F 3 "~" H 6450 3550 50  0001 C CNN
+	1    6450 3550
+	1    0    0    -1
+$EndComp
+$Comp
+L Device:C c9
+U 1 1 607578C6
+P 8350 3850
+F 0 "c9" H 8465 3896 50  0000 L CNN
+F 1 "100n" H 8465 3805 50  0000 L CNN
+F 2 "Capacitor_SMD:C_0805_2012Metric_Pad1.18x1.45mm_HandSolder" H 8388 3700 50  0001 C CNN
+F 3 "~" H 8350 3850 50  0001 C CNN
+	1    8350 3850
+	1    0    0    -1
+$EndComp
+Wire Wire Line
+	6450 3700 6750 3700
+Connection ~ 6750 3700
+Wire Wire Line
+	8350 4000 8500 4000
+Connection ~ 8500 4000
+Wire Wire Line
+	8500 4000 8500 4050
+$Comp
+L power:GND #PWR086
+U 1 1 6077B10C
+P 8350 3700
+F 0 "#PWR086" H 8350 3450 50  0001 C CNN
+F 1 "GND" H 8355 3527 50  0000 C CNN
+F 2 "" H 8350 3700 50  0001 C CNN
+F 3 "" H 8350 3700 50  0001 C CNN
+	1    8350 3700
+	-1   0    0    1
+$EndComp
+$Comp
+L power:GND #PWR085
+U 1 1 6077B39F
+P 6450 3400
+F 0 "#PWR085" H 6450 3150 50  0001 C CNN
+F 1 "GND" H 6455 3227 50  0000 C CNN
+F 2 "" H 6450 3400 50  0001 C CNN
+F 3 "" H 6450 3400 50  0001 C CNN
+	1    6450 3400
+	-1   0    0    1
+$EndComp
+Wire Wire Line
+	4200 2100 4350 2100
+$Comp
+L Device:C c1
+U 1 1 607B67B0
+P 4350 2250
+F 0 "c1" H 4465 2296 50  0000 L CNN
+F 1 "100n" H 4465 2205 50  0000 L CNN
+F 2 "Capacitor_SMD:C_0805_2012Metric_Pad1.18x1.45mm_HandSolder" H 4388 2100 50  0001 C CNN
+F 3 "~" H 4350 2250 50  0001 C CNN
+	1    4350 2250
+	1    0    0    -1
+$EndComp
+Connection ~ 4350 2100
+Wire Wire Line
+	4350 2100 4700 2100
 $EndSCHEMATC

Commit message: hardware done
Parts:
- added R36: 50k, Potentiometers:Potentiometer_Trimmer_Bourns_3296W, symbol Device:RTRIM
- R27: value 1.5k -> 22k
Connections:
- wire segments 236 -> 241
Other:
- note added: "LP\n"
- note removed: "11 khz LP\n"
- moved on the sheet: c7
Changed lines of the file:
@@
 P 9450 4450
 F 0 "R27" V 9243 4450 50  0000 C CNN
-F 1 "1.5k" V 9334 4450 50  0000 C CNN
+F 1 "22k" V 9334 4450 50  0000 C CNN
 F 2 "Resistor_SMD:R_0805_2012Metric_Pad1.20x1.40mm_HandSolder" V 9380 4450 50  0001 C CNN
 F 3 "~" H 9450 4450 50  0001 C CNN
@@
 L Device:C c7
 U 1 1 6053A73E
-P 9650 4650
-F 0 "c7" H 9765 4696 50  0000 L CNN
-F 1 "10n" H 9500 4550 50  0000 L CNN
-F 2 "Capacitor_SMD:C_0805_2012Metric_Pad1.18x1.45mm_HandSolder" H 9688 4500 50  0001 C CNN
-F 3 "~" H 9650 4650 50  0001 C CNN
-	1    9650 4650
-	1    0    0    -1
-$EndComp
-Wire Wire Line
-	9650 4500 9650 4450
-Wire Wire Line
-	9600 4450 9650 4450
-Connection ~ 9650 4450
-Wire Wire Line
-	9650 4450 9850 4450
-Wire Wire Line
-	9200 4450 9300 4450
+P 9650 5100
+F 0 "c7" H 9765 5146 50  0000 L CNN
+F 1 "10n" H 9500 5000 50  0000 L CNN
+F 2 "Capacitor_SMD:C_0805_2012Metric_Pad1.18x1.45mm_HandSolder" H 9688 4950 50  0001 C CNN
+F 3 "~" H 9650 5100 50  0001 C CNN
+	1    9650 5100
+	1    0    0    -1
+$EndComp
+Wire Wire Line
+	9200 4450 9250 4450
 $Comp
 L power:GND #PWR066
 U 1 1 60544749
-P 9650 4800
-F 0 "#PWR066" H 9650 4550 50  0001 C CNN
-F 1 "GND" H 9655 4627 50  0000 C CNN
-F 2 "" H 9650 4800 50  0001 C CNN
-F 3 "" H 9650 4800 50  0001 C CNN
-	1    9650 4800
+P 9650 5250
+F 0 "#PWR066" H 9650 5000 50  0001 C CNN
+F 1 "GND" H 9655 5077 50  0000 C CNN
+F 2 "" H 9650 5250 50  0001 C CNN
+F 3 "" H 9650 5250 50  0001 C CNN
+	1    9650 5250
 	1    0    0    -1
 $EndComp
@@
 	9500 4100 10450 4100
 Text Notes 9200 4600 0    50   ~ 0
-11 khz LP\n
+LP\n
 $Comp
 L Device:R_POT P_A1
@@
 	7500 600  9450 600
 Connection ~ 9450 600
-$Comp
-L Device:LED D4
-U 1 1 605EC90A
-P 11400 2650
-F 0 "D4" V 11439 2730 50  0000 L CNN
-F 1 "LED" V 11348 2730 50  0000 L CNN
-F 2 "LED_THT:LED_D5.0mm" H 11400 2650 50  0001 C CNN
-F 3 "~" H 11400 2650 50  0001 C CNN
-	1    11400 2650
-	0    1    -1   0
-$EndComp
 Text Notes 11850 2650 0    50   ~ 0
 outLED\n
@@
 	0    1    1    0
 $EndComp
-Connection ~ 10550 2800
-Wire Wire Line
-	10550 2800 11400 2800
-Wire Wire Line
-	11400 2500 10550 2500
 Wire Wire Line
 	10550 2500 9850 2500
 Wire Wire Line
 	9850 2500 9850 2700
-Connection ~ 10550 2500
 Wire Wire Line
 	9500 2700 9500 3650
@@
 Wire Wire Line
 	4350 2100 4700 2100
+$Comp
+L Device:RTRIM R36
+U 1 1 6055E0DB
+P 9450 4850
+F 0 "R36" V 9715 4850 50  0000 C CNN
+F 1 "50k" V 9624 4850 50  0000 C CNN
+F 2 "Potentiometers:Potentiometer_Trimmer_Bourns_3296W" V 9380 4850 50  0001 C CNN
+F 3 "~" H 9450 4850 50  0001 C CNN
+	1    9450 4850
+	0    -1   -1   0
+$EndComp
+Wire Wire Line
+	9600 4450 9650 4450
+Wire Wire Line
+	9650 4450 9650 4850
+Connection ~ 9650 4450
+Wire Wire Line
+	9650 4450 9850 4450
+Wire Wire Line
+	9600 4850 9650 4850
+Connection ~ 9650 4850
+Wire Wire Line
+	9650 4850 9650 4950
+Wire Wire Line
+	9300 4850 9250 4850
+Wire Wire Line
+	9250 4850 9250 4450
+Connection ~ 9250 4450
+Wire Wire Line
+	9250 4450 9300 4450
+Connection ~ 10550 2500
+Connection ~ 10550 2800
+Wire Wire Line
+	11400 2500 10550 2500
+Wire Wire Line
+	10550 2800 11400 2800
+$Comp
+L Device:LED D4
+U 1 1 605EC90A
+P 11400 2650
+F 0 "D4" V 11439 2730 50  0000 L CNN
+F 1 "LED" V 11348 2730 50  0000 L CNN
+F 2 "LED_THT:LED_D5.0mm" H 11400 2650 50  0001 C CNN
+F 3 "~" H 11400 2650 50  0001 C CNN
+	1    11400 2650
+	0    1    -1   0
+$EndComp
 $EndSCHEMATC
