File: hardware/ADSR_frontpanel.kicad_pcb (KiCad board)
At the start: 2 copper layers, 91.4 x 129.5 mm, 0 parts

Commit message: hardware done
Parts:
- added G***: LOGO, hardware:KP_logo, F.Cu at (178.5, 136.8)
Other:
- board size 91.4 x 129.5 mm -> 91.4 x 128.5 mm
